Commit message: works

File: resource/spot.urdf (robot description, URDF)
Before this commit: robot Spot, 78 links, 77 joints
Links:
- removed link SpotArm
- removed link cap screw
- removed link cap screw(1)
- removed link cap screw(10)
- removed link cap screw(11)
- removed link cap screw(12)
- removed link cap screw(13)
- removed link cap screw(14)
- removed link cap screw(15)
- removed link cap screw(16)
- removed link cap screw(17)
- removed link cap screw(18)
- removed link cap screw(19)
- removed link cap screw(2)
- removed link cap screw(3)
- removed link cap screw(4)
- removed link cap screw(5)
- removed link cap screw(6)
- removed link cap screw(7)
- removed link cap screw(8)
- removed link cap screw(9)
- removed link front
- removed link gripper_centre
- removed link gripper_left_finger_link
- removed link gripper_right_finger_link
- removed link spotarm_link1
- removed link spotarm_link2
- removed link spotarm_link3
- removed link spotarm_link4
- removed link spotarm_link5
- removed link spotarm_link6
- added link lidar; collision cylinder length=0.0727 radius=0.052; visual cylinder length=0.0727 radius=0.052
Joints:
- removed joint Slider11
- removed joint base_link_SpotArm_joint
- removed joint front_cap screw(1)_joint
- removed joint front_cap screw(10)_joint
- removed joint front_cap screw(11)_joint
- removed joint front_cap screw(12)_joint
- removed joint front_cap screw(13)_joint
- removed joint front_cap screw(14)_joint
- removed joint front_cap screw(15)_joint
- removed joint front_cap screw(16)_joint
- removed joint front_cap screw(17)_joint
- removed joint front_cap screw(18)_joint
- removed joint front_cap screw(19)_joint
- removed joint front_cap screw(2)_joint
- removed joint front_cap screw(3)_joint
- removed joint front_cap screw(4)_joint
- removed joint front_cap screw(5)_joint
- removed joint front_cap screw(6)_joint
- removed joint front_cap screw(7)_joint
- removed joint front_cap screw(8)_joint
- removed joint front_cap screw(9)_joint
- removed joint front_cap screw_joint
- removed joint gripper_centre_joint
- removed joint gripper_left_finger_joint
- removed joint gripper_right_finger_joint
- removed joint spotarm_1_joint
- removed joint spotarm_2_joint
- removed joint spotarm_3_joint
- removed joint spotarm_4_joint
- removed joint spotarm_5_joint
- removed joint spotarm_6_joint
- added joint base_link_lidar_joint: type fixed, parent base_link, child lidar, origin xyz=-0.063 0 0.1518 rpy=-0.000008 -0.000008 0.000001

Commit message: zx

File: resource/spot.urdf (robot description, URDF)
Before this commit: robot Spot, 48 links, 47 joints
Joints:
- joint base_link_lidar_joint: origin xyz=-0.063 0 0.1518 rpy=-0.000008 -0.000008 0.000001 -> xyz=-0.13 0 0.1518 rpy=-0.000008 -0.000008 0.000001
